Commit message: Updates

File: piper_ros/src/piper_description/urdf/piper_description.xacro (robot description, xacro)
@@ -8,4 +8,5 @@
       <parent link="world"/>
       <child link="base_link"/>
+      <origin xyz="0 0 0.33" rpy="0 0 0"/>
   </joint>
 <!-- arm -->
@@ -336,4 +337,31 @@
       effort="100"
       velocity="3" />
+  </joint>
+  <link name="d435i_link">
+    <visual>
+      <origin xyz="0 0 0" rpy="0 0 0" />
+      <geometry>
+          <mesh filename="package://piper_description/meshes/D435i.STL" scale="0.001 0.001 0.001"/>
+      </geometry>
+      <material name="gray">
+        <color rgba="0.3 0.3 0.3 1"/>
+      </material>
+    </visual>
+    <collision>
+      <origin xyz="0 0 0" rpy="0 0 0" />
+      <geometry>
+          <mesh filename="package://piper_description/meshes/D435i.STL" scale="0.001 0.001 0.001"/>
+      </geometry>
+    </collision>
+    <inertial>
+      <origin xyz="0 0 0" rpy="0 0 0"/>
+      <mass value="0.072"/>
+      <inertia ixx="1e-5" ixy="0" ixz="0" iyy="1e-5" iyz="0" izz="1e-5"/>
+    </inertial>
+  </link>
+  <joint name="link6_to_d435i" type="fixed">
+    <origin xyz="-0.045 -0.045 0.05" rpy="0 0 1.5708"/>
+    <parent link="link6"/>
+    <child link="d435i_link"/>
   </joint>
   <link

File: piper_ros/src/piper_moveit/piper_with_gripper_moveit/config/piper.ros2_control.xacro (robot description, xacro)
@@ -1,14 +1,19 @@
 <?xml version="1.0"?>
 <robot xmlns:xacro="http://www.ros.org/wiki/xacro">
-    <xacro:macro name="piper_ros2_control" params="name initial_positions_file">
+    <xacro:macro name="piper_ros2_control" params="name initial_positions_file real">
+    <!-- <xacro:macro name="piper_ros2_control" params="name initial_positions_file"> -->
         <xacro:property name="initial_positions" value="${load_yaml(initial_positions_file)['initial_positions']}"/>
         <ros2_control name="${name}" type="system">
             <hardware>
               <!-- for Real -->
-              <plugin>topic_based_ros2_control/TopicBasedSystem</plugin>
-              <param name="joint_commands_topic">/joint_ctrl_single</param>
-              <param name="joint_states_topic">/joint_states</param>
+              <xacro:if value="${real}">
+                <plugin>topic_based_ros2_control/TopicBasedSystem</plugin>
+                <param name="joint_commands_topic">/joint_ctrl_single</param>
+                <param name="joint_states_topic">/joint_states</param>
+              </xacro:if>
               <!-- for Sim -->
-              <!-- <plugin>mock_components/GenericSystem</plugin> -->
+              <xacro:unless value="${real}">
+                <plugin>mock_components/GenericSystem</plugin>
+              </xacro:unless>
             </hardware>
             <joint name="joint1">

File: piper_ros/src/piper_moveit/piper_with_gripper_moveit/config/piper.urdf.xacro (robot description, xacro)
@@ -2,8 +2,10 @@
 <robot xmlns:xacro="http://www.ros.org/wiki/xacro" name="piper">
     <xacro:arg name="initial_positions_file" default="initial_positions.yaml" />
+    <xacro:arg name="real" default="false" />
     <!-- Import piper urdf file -->
     <xacro:include filename="$(find piper_description)/urdf/piper_description.xacro" />
     <!-- Import control_xacro -->
     <xacro:include filename="piper.ros2_control.xacro" />
-    <xacro:piper_ros2_control name="FakeSystem" initial_positions_file="$(arg initial_positions_file)"/>
+    <xacro:piper_ros2_control name="FakeSystem" initial_positions_file="$(arg initial_positions_file)" real="$(arg real)"/>
+    <!-- <xacro:piper_ros2_control name="FakeSystem" initial_positions_file="$(arg initial_positions_file)" real="$(arg real)"/> -->
 </robot>

Commit message: change wm

File: piper_ros/src/piper_description/urdf/piper_description.xacro (robot description, xacro)
@@ -8,5 +8,5 @@
       <parent link="world"/>
       <child link="base_link"/>
-      <origin xyz="0 0 0.33" rpy="0 0 0"/>
+      <origin xyz="0 0 0.37" rpy="0 0 0"/>
   </joint>
 <!-- arm -->
